File: K9HZ_LPF_Module/K9HZ_LPF_V1.00_Schematics/K9HZ_100W_11band_LPF-Control/K9HZ_100W_11band_LPF-Control.kicad_sch (KiCad schematic)
At the start: 155 parts, among them J1 LPF ACC Control, J10 FROM 100W PA, J11 ANT-1, J12 ANT-2, J13 ANT-3, J14 ANT-4, J15 TO BPF, J16 TO LPF, J16.1 ANTENNA, J16.2 TRANSMIT, J17.1 RECEIVE, J17.2 TR CTL, J18 FROM BPF, J19 KEY OUT, J2 TO_RECEIVER, J20 12-13.8V, J21 Bands, J23 FROM LPF, J24 LPF CTRL HI, J25 LPF CTRL LOW, J3 FROM TX, J4 TO ATTN, J5 FROM ATTN, J6 TO XVTR, J7 TO 20W PA, J8 FROM 20W PA, J9 TO 100W PA, K2 HF41F/12-ZS, K3 HF41F/12-ZS, K4 HF41F/12-ZS, K5 HF41F/12-ZS, K6 HF41F/12-ZS, K7 HF41F/12-ZS, Q1 IRF630, Q2 2N7000, U1 MASWSS0179, U10 ULN2803C, U11 LM7805CT, U12 CD74HC4514M96, U13 L7808, U14 AD8307, U15 MCP23017_SO, U16 LM1117T-3.3, U17 REF3440IDBVR, U18 TC4428, U19 AD8307, U2 74HC237, U20 AD7991YRJZ, U21 MASWSS0179, U22 SN74LVC1G04DCK, U3 MASWSS0179, U4 ULN2803C, U5 SN74LVC1G04DCK, U6 SN74LVC1G04DCK, U7 MASWSS0179, U8 MASWSS0179, U9 ULN2803C

Commit message: Fixed missing connection between pins 5 and 6 on U17, REF3440
Connections:
- net at U17.5 (OUT_S): now also C145.1, U17.6 (OUT_F), U20.6 (Vin3/Vref)
- no-connect marks 43 -> 42
