File: K9HZ_Antenna_Tuner/K9HZ_100W_Antenna_Tuner_V1.10/K9HZ_100W_Antenna_Tuner_V1.10.kicad_pcb (KiCad board)
At the start: 2 copper layers, 8 parts, among them J11 SOLDER_JMP_2, U1 MCP23017_SO, U2 UDN2987LW, U3 MCP23008-E/SO, U4 UDN2987LW, U5 UDN2987LW

Commit message: Update Files
Update Files
Parts:
- added J11: SOLDER_JMP_2, Jumper:SolderJumper-2_P1.3mm_Open_RoundedPad1.0x1.5mm, F.Cu at (85.7, 152.4)
- moved U5 65.9 mm to (114.3, 88.9)
- moved U3 64.3 mm to (114.3, 132.1)
- moved U4 56.2 mm to (88.9, 88.9), turned to -90 degrees
- moved C17 24.0 mm to (96.5, 142.2), turned to 180 degrees
- moved C13 22.7 mm to (99.1, 119.4), turned to 180 degrees
- moved J11 20.4 mm to (118.7, 152.4)
- moved U2 8.27 mm to (91.4, 132.1), turned to 90 degrees
- turned U1 to -90 degrees
