File: K9HZ_Antenna_Tuner/K9HZ_100W_Antenna_Tuner_V1.10/K9HZ_100W_Antenna_Tuner_V1.10.kicad_sch (KiCad schematic)
At the start: 71 parts, among them J1 901-144, J10 SOLDER_JMP_2, J11 SOLDER_JMP_2, J2 901-144, J20 395310002, J5 BANDS, J6 SOLDER_JMP_2, J7 SOLDER_JMP_2, J8 SOLDER_JMP_2, J9 SOLDER_JMP_2, K1 HF41F-12-ZS, K10 HF41F-12-ZS, K11 HF41F-12-ZS, K12 HF41F-12-ZS, K13 HF41F-12-ZS, K14 HF41F-12-ZS, K15 HF41F-12-ZS, K16 HF41F-12-ZS, K17 HF41F-12-ZS, K18 HF41F-12-ZS_10, K19 HF41F-12-ZS, K2 HF41F-12-ZS, K20 HF41F-12-ZS_11, K3 HF41F-12-ZS, K4 HF41F-12-ZS, K5 HF41F-12-ZS, K6 HF41F-12-ZS, K7 HF41F-12-ZS, K8 HF41F-12-ZS, K9 HF41F-12-ZS, T1 1T 4, U1 MCP23017_SO, U2 UDN2987LW, U3 MCP23008-E/SO, U4 UDN2987LW, U5 UDN2987LW, U6 L7805ABD2T-TR

Commit message: Update Files
Update Files
Connections:
- net +5V: now also C18.1 (PLUS)
- net at K18.NC: now also J2.5 (CON)
- net at K18.NO: no longer T1.1
- net at U1.13 (SDA), U3.2 (SDA): now also J5.5 (P5)
- now unconnected: K18.C (COM), K20.C (COM)
Other:
- title: (none) -> K9HZ 100W Antenna Tuner for T41 V12
- moved on the sheet: J10
