File: K9HZ_LPF_Module/K9HZ_LPF_Schematics/K9HZ_100W_11band_LPF-TR-carrier/K9HZ_100W_11band_LPF-TR-carrier_01_06_26.kicad_pcb (KiCad board)
At the start: 2 copper layers, 40.6 x 25.4 mm, 12 parts, among them J22.1 ANTENNA, J22.2 TRANSMIT, J23.1 RECEIVE, J23.2 TR CTL, K1 HF41F/12-ZS, K2 HF41F/12-ZS, Q1 BS170

Commit message: ATU Update
ATU Update
Parts:
- added ?: , , F.Cu at (115.1, 79.0)
- added ?: , , F.Cu at (64.0, 83.8)
- added ?: , , F.Cu at (115.1, 84.1)
- added ?: , , F.Cu at (69.1, 78.7)
- added ?: , , F.Cu at (120.1, 84.1)
- added ?: , , F.Cu at (120.1, 79.0)
- added ?: , , F.Cu at (117.6, 81.5)
- added ?: , , F.Cu at (69.1, 83.8)
- added ?: , , F.Cu at (66.5, 81.3)
- added ?: , , F.Cu at (64.0, 78.7)
Connections:
- K1 pad 12: /ANT -> (no net)
- K2 pad 14: /ANT -> (no net)
Routing:
- net /ANT: track 22.6 -> 59.4 mm
- net GND: vias 55 -> 57

Commit message: Updates for Tuner
Updates for Tuner
Routing:
- net (no net): track 0.00 -> 41.9 mm
- net /ANT: track 59.4 -> 19.2 mm
Other:
- board size 40.6 x 25.4 mm -> 61.5 x 25.4 mm
- board text added: "FROM TUNER"
- board text added: "TO TUNER"
Changed lines of the file:
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@@
 			(outputformat 1)
 			(mirror no)
-			(drillshape 1)
+			(drillshape 0)
 			(scaleselection 1)
-			(outputdirectory "")
+			(outputdirectory "Gerber Files/")
 		)
 	)
@@
 		(embedded_fonts no)
 	)
-	(gr_rect
-		(start 71.755 76.2)
-		(end 112.395 101.6)
+	(gr_poly
+		(pts
+			(xy 71.628 86.36) (xy 61.468 86.36) (xy 61.468 76.2) (xy 122.936 76.2) (xy 122.936 86.614) (xy 112.522 86.614)
+			(xy 112.522 101.6) (xy 71.628 101.6)
+		)
 		(stroke
 			(width 0.1)
-			(type default)
+			(type solid)
 		)
 		(fill no)
@@
 		)
 	)
+	(gr_text "FROM TUNER"
+		(at 112.776 77.724 0)
+		(layer "F.SilkS")
+		(effects
+			(font
+				(size 1 1)
+				(thickness 0.15)
+			)
+			(justify left bottom)
+		)
+	)
 	(gr_text "TR CTL"
 		(at 90.3732 97.536 0)
@@
 		)
 	)
+	(gr_text "TO TUNER"
+		(at 63.246 77.724 0)
+		(layer "F.SilkS")
+		(effects
+			(font
+				(size 1 1)
+				(thickness 0.15)
+			)
+			(justify left bottom)
+		)
+	)
 	(gr_text "TR Switch Carrier\n2026/01/06"
 		(at 72.898 79.248 0)
@@
 		)
 	)
+	(segment
+		(start 72.644 79.756)
+		(end 83.312 79.756)
+		(width 0.525)
+		(layer "F.Cu")
+		(net 0)
+	)
+	(segment
+		(start 83.312 79.756)
+		(end 86.741 83.185)
+		(width 0.525)
+		(layer "F.Cu")
+		(net 0)
+	)
+	(segment
+		(start 96.393 85.598)
+		(end 100.758 85.598)
+		(width 0.525)
+		(layer "F.Cu")
+		(net 0)
+	)
+	(segment
+		(start 86.741 83.185)
+		(end 93.98 83.185)
+		(width 0.525)
+		(layer "F.Cu")
+		(net 0)
+	)
+	(segment
+		(start 93.98 83.185)
+		(end 96.393 85.598)
+		(width 0.525)
+		(layer "F.Cu")
+		(net 0)
+	)
+	(segment
+		(start 71.12 81.28)
+		(end 72.644 79.756)
+		(width 0.525)
+		(layer "F.Cu")
+		(net 0)
+	)
+	(segment
+		(start 100.758 85.598)
+		(end 104.06 88.9)
+		(width 0.525)
+		(layer "F.Cu")
+		(net 0)
+	)
+	(segment
+		(start 66.548 81.28)
+		(end 71.12 81.28)
+		(width 0.525)
+		(layer "F.Cu")
+		(net 0)
+	)
 	(via
 		(at 102.616 91.694)
@@
 		(drill 0.4)
 		(layers "F.Cu" "B.Cu")
-		(free yes)
 		(net 1)
 	)
@@
 		(drill 0.4)
 		(layers "F.Cu" "B.Cu")
-		(free yes)
 		(net 1)
 	)
 	(via
-		(at 88.4428 83.9724)
+		(at 88.138 84.836)
 		(size 0.8)
 		(drill 0.4)
@@
 		(drill 0.4)
 		(layers "F.Cu" "B.Cu")
-		(free yes)
 		(net 1)
 	)
@@
 	)
 	(segment
-		(start 84.0635 94.1035)
-		(end 78.86 88.9)
+		(start 90.297 93.472)
+		(end 83.432 93.472)
 		(width 0.293)
 		(layer "B.Cu")
@@
 	)
 	(segment
-		(start 92.075 95.25)
-		(end 90.9285 94.1035)
+		(start 83.432 93.472)
+		(end 78.86 88.9)
 		(width 0.293)
 		(layer "B.Cu")
@@
 	)
 	(segment
-		(start 90.9285 94.1035)
-		(end 84.0635 94.1035)
+		(start 78.86 88.9)
+		(end 78.86 83.185)
 		(width 0.293)
 		(layer "B.Cu")
@@
 	)
 	(segment
-		(start 78.86 88.9)
-		(end 78.86 83.185)
+		(start 92.075 95.25)
+		(end 90.297 93.472)
 		(width 0.293)
 		(layer "B.Cu")
@@
 	)
 	(segment
-		(start 96.5708 85.7758)
-		(end 93.98 83.185)
-		(width 0.525)
-		(layer "F.Cu")
-		(net 5)
-	)
-	(segment
-		(start 66.548 81.28)
-		(end 71.628 81.28)
-		(width 0.525)
-		(layer "F.Cu")
-		(net 5)
-	)
-	(segment
-		(start 83.82 80.01)
-		(end 86.106 82.296)
-		(width 0.525)
-		(layer "F.Cu")
-		(net 5)
-	)
-	(segment
-		(start 73.66 80.01)
-		(end 83.82 80.01)
-		(width 0.525)
-		(layer "F.Cu")
-		(net 5)
-	)
-	(segment
-		(start 104.06 88.9)
-		(end 100.9358 85.7758)
-		(width 0.525)
-		(layer "F.Cu")
-		(net 5)
-	)
-	(segment
 		(start 109.855 83.82)
 		(end 109.855 86.36)
@@
 	)
 	(segment
-		(start 72.136 81.534)
-		(end 73.66 80.01)
-		(width 0.525)
-		(layer "F.Cu")
-		(net 5)
-	)
-	(segment
 		(start 109.855 83.82)
-		(end 109.982 83.82)
+		(end 109.855 83.185)
 		(width 0.525)
 		(layer "F.Cu")
@@
 	)
 	(segment
-		(start 86.106 82.296)
-		(end 93.091 82.296)
+		(start 111.506 81.534)
+		(end 117.602 81.534)
 		(width 0.525)
 		(layer "F.Cu")
@@
 	)
 	(segment
-		(start 117.602 81.534)
-		(end 112.776 81.534)
-		(width 0.525)
-		(layer "F.Cu")
-		(net 5)
-	)
-	(segment
-		(start 93.091 82.296)
-		(end 93.98 83.185)
-		(width 0.525)
-		(layer "F.Cu")
-		(net 5)
-	)
-	(segment
-		(start 100.9358 85.7758)
-		(end 96.5708 85.7758)
+		(start 109.855 83.185)
+		(end 111.506 81.534)
 		(width 0.525)
 		(layer "F.Cu")
@@
 	)
 	(segment
-		(start 72.0185 81.534)
-		(end 72.136 81.534)
-		(width 0.525)
-		(layer "F.Cu")
-		(net 5)
-	)
-	(segment
-		(start 109.982 83.82)
-		(end 112.014 81.788)
-		(width 0.525)
-		(layer "F.Cu")
-		(net 5)
-	)
-	(segment
 		(start 74.295 88.9)
 		(end 74.295 91.44)
@@
 		(min_thickness 0.25)
 		(filled_areas_thickness no)
-		(fill
-			(thermal_gap 0.5)
-			(thermal_bridge_width 0.5)
-			(island_removal_mode 1)
-			(island_area_min 10)
-		)
-		(polygon
-			(pts
-				(xy 61.468 76.2) (xy 61.468 86.36) (xy 71.755 86.36) (xy 71.755 76.2)
-			)
-		)
-	)
-	(zone
-		(net 1)
-		(net_name "GND")
-		(layers "F.Cu" "B.Cu")
-		(hatch edge 0.5)
-		(connect_pads
-			(clearance 0.5)
-		)
-		(min_thickness 0.25)
-		(filled_areas_thickness no)
-		(fill
-			(thermal_gap 0.5)
-			(thermal_bridge_width 0.5)
-		)
-		(polygon
-			(pts
-				(xy 112.395 76.2) (xy 122.936 76.2) (xy 122.936 86.614) (xy 112.395 86.614)
-			)
-		)
-	)
-	(zone
-		(net 1)
-		(net_name "GND")
-		(layers "F.Cu" "B.Cu")
-		(hatch edge 0.5)
-		(connect_pads
-			(clearance 0.5)
-		)
-		(min_thickness 0.25)
-		(filled_areas_thickness no)
 		(fill yes
 			(thermal_gap 0.5)
@@
 		(polygon
 			(pts
-				(xy 71.755 76.2) (xy 112.395 76.2) (xy 112.395 101.6) (xy 71.755 101.6)
+				(xy 61.468 76.2) (xy 61.468 86.36) (xy 71.628 86.36) (xy 71.628 101.6) (xy 112.522 101.6) (xy 112.522 86.614)
+				(xy 122.936 86.614) (xy 122.936 76.2)
 			)
 		)
