File: K9HZ_Antenna_Tuner/K9HZ_Antenna_Tuner_KiCad_Projects/K9HZ_Antenna_Tuner_Control_Board_Project/K9HZ_Antenna_Tuner_Control_Board.kicad_sch (KiCad schematic)
At the start: 67 parts, among them J1 1986717-8, J10 IDC2x5, J11 395310002, J2 1986717-8, J3 1986717-8, J4 A0, J5 A1, J6 A2, J7 A0, J8 A1, J9 A2, U1 L7805ABD2T-TR, U2 UDN2987LWTR-6-T, U3 UDN2987LWTR-6-T, U4 UDN2987LWTR-6-T, U5 MCP23017_SO, U6 MCP23008-E/SO

Commit message: Tuner Update
Tuner Update
Parts:
- removed R11, R8: 52.3, Resistor_SMD:R_1206_3216Metric_Pad1.30x1.75mm_HandSolder, symbol Device:R_US
Other:
- note added: "LINE SECTION OPTION: NOT USED FOR T41 WITH LPF LINE SECTION"
