File: K9HZ_Antenna_Tuner/K9HZ_Antenna_Tuner_KiCad_Projects/K9HZ_Antenna_Tuner_Control_Board_Project/K9HZ_Antenna_Tuner_Control_Board.kicad_pcb (KiCad board)
At the start: 2 copper layers, 71.5 x 81.2 mm, 67 parts, among them J1 1986717-8, J10 IDC2x5, J11 395310002, J2 1986717-8, J3 1986717-8, J4 A0, J5 A1, J6 A2, J7 A0, J8 A1, J9 A2, U1 L7805ABD2T-TR, U2 UDN2987LWTR-6-T, U3 UDN2987LWTR-6-T, U4 UDN2987LWTR-6-T, U5 MCP23017_SO, U6 MCP23008-E/SO

Commit message: Tuner Update
Tuner Update
Parts:
- removed R11, R8: 52.3, Resistor_SMD:R_1206_3216Metric_Pad1.30x1.75mm_HandSolder
- J10, J11, VR1, VR2: moved to B.Cu
- moved J10 85.2 mm to (112.1, 106.5)
- moved U1 81.0 mm to (115.2, 82.1)
- moved VR1 80.2 mm to (123.3, 124.1), turned to -90 degrees
- moved VR2 80.2 mm to (113.9, 124.1), turned to -90 degrees
- moved C21 79.6 mm to (118.4, 68.4)
- moved C20 78.0 mm to (133.8, 76.2)
- moved C23 78.0 mm to (155.8, 122.0)
- moved C27 78.0 mm to (142.5, 107.0)
- moved C28 78.0 mm to (136.5, 73.7)
- moved R1 78.0 mm to (132.0, 80.8)
- moved R2 78.0 mm to (132.0, 83.8)
- moved R4 78.0 mm to (134.8, 101.2)
- moved U6 78.0 mm to (132.8, 110.8)
- moved C1 78.0 mm to (167.7, 111.7)
- moved C10 78.0 mm to (167.7, 103.1)
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Connections:
- J10 pad 1: unconnected-(J10-Pin_1-Pad1) -> (no net)
- J10 pad 10: unconnected-(J10-Pin_10-Pad10) -> (no net)
- J10 pad 2: unconnected-(J10-Pin_2-Pad2) -> (no net)
- J10 pad 3: unconnected-(J10-Pin_3-Pad3) -> (no net)
- J10 pad 4: unconnected-(J10-Pin_4-Pad4) -> (no net)
- J11 pad 1: GND -> +12V
- J11 pad 2: +12V -> GND
- VR1 pad 1: GND -> Net-(D1-(C))
- VR1 pad 3: Net-(D1-(C)) -> GND
- VR2 pad 1: GND -> Net-(D2-(C))
- VR2 pad 3: Net-(D2-(C)) -> GND
Routing:
- net +12V: track 104.1 -> 113.6 mm
- net Net-(J10-Pin_5): track 68.8 -> 77.8 mm
- net Net-(J10-Pin_7): track 66.8 -> 73.0 mm
- net Net-(J10-Pin_8): track 20.8 -> 24.8 mm
- net Net-(J10-Pin_6): track 23.2 -> 20.4 mm, vias 0 -> 1
- net Net-(D1-(A)): track 32.6 -> 31.3 mm
- net +5V: track 186.5 -> 187.5 mm
- net Net-(U2-IN8): track 12.2 -> 11.3 mm
- net Net-(U2-IN7): track 12.9 -> 12.1 mm
- net GND: track 3.60 -> 4.08 mm, vias 2 -> 320
Other:
- board size 71.5 x 81.2 mm -> 70.9 x 81.2 mm
- board text added: "BANDS"
- board text added: "NC"
- board text added: "SCL"
- board text added: "SDA"

Commit message: Update Tuner
Update Tuner for Production
Routing:
- net (no net): track 0.00 -> 51.6 mm
- net GND: vias 320 -> 316

Commit message: Antenna Tuner Update
Antenna Tuner Update
Routing:
- net GND: track 4.08 -> 55.6 mm
- net (no net): track 51.6 -> 0.00 mm
Changed lines of the file:
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@@
 			(drillshape 0)
 			(scaleselection 1)
-			(outputdirectory "")
+			(outputdirectory "C:/Users/Dad/Documents/GitHub/K9HZ/K9HZ_Antenna_Tuner/K9HZ_Antenna_Tuner_Gerbers/")
 		)
 	)
@@
 	)
 	(segment
-		(start 106.144 88.396)
-		(end 106.144 88.543)
-		(width 0.2)
-		(layer "B.Cu")
-		(net 0)
-	)
-	(segment
-		(start 115.86 88.56)
-		(end 115.843 88.543)
-		(width 0.2)
-		(layer "B.Cu")
-		(net 0)
-	)
-	(segment
-		(start 116.496 88.394057)
-		(end 116.330057 88.56)
-		(width 0.2)
-		(layer "B.Cu")
-		(net 0)
-	)
-	(segment
-		(start 115.843 88.543)
-		(end 114.792943 88.543)
-		(width 0.6)
-		(layer "B.Cu")
-		(net 0)
-	)
-	(segment
-		(start 116.68 77.02)
-		(end 116.496 77.204)
-		(width 0.2)
-		(layer "B.Cu")
-		(net 0)
-	)
-	(segment
-		(start 116.330057 88.56)
-		(end 115.86 88.56)
-		(width 0.6)
-		(layer "B.Cu")
-		(net 0)
-	)
-	(segment
-		(start 106.144 88.396)
-		(end 106.14 88.4)
-		(width 0.2)
-		(layer "B.Cu")
-		(net 0)
-	)
-	(segment
-		(start 116.496 82.142)
-		(end 116.496 88.394057)
-		(width 0.6)
-		(layer "B.Cu")
-		(net 0)
-	)
-	(segment
-		(start 116.496 75.741)
-		(end 106.144 75.741)
-		(width 0.6)
-		(layer "B.Cu")
-		(net 0)
-	)
-	(segment
-		(start 106.144 88.543)
-		(end 114.92 88.543)
-		(width 0.6)
-		(layer "B.Cu")
-		(net 0)
-	)
-	(segment
-		(start 116.496 82.142)
-		(end 116.496 75.741)
-		(width 0.6)
-		(layer "B.Cu")
-		(net 0)
-	)
-	(segment
-		(start 116.496 77.204)
-		(end 116.496 82.142)
-		(width 0.2)
-		(layer "B.Cu")
-		(net 0)
-	)
-	(segment
-		(start 106.144 75.741)
-		(end 106.144 88.396)
-		(width 0.6)
-		(layer "B.Cu")
-		(net 0)
-	)
-	(segment
 		(start 152.973 121.475)
 		(end 154.8005 121.475)
@@
 		(net 1)
 	)
+	(segment
+		(start 106.144 88.396)
+		(end 106.144 88.543)
+		(width 0.2)
+		(layer "B.Cu")
+		(net 1)
+	)
+	(segment
+		(start 115.86 88.56)
+		(end 115.843 88.543)
+		(width 0.2)
+		(layer "B.Cu")
+		(net 1)
+	)
+	(segment
+		(start 116.496 88.394057)
+		(end 116.330057 88.56)
+		(width 0.2)
+		(layer "B.Cu")
+		(net 1)
+	)
+	(segment
+		(start 115.843 88.543)
+		(end 114.792943 88.543)
+		(width 1.5)
+		(layer "B.Cu")
+		(net 1)
+	)
+	(segment
+		(start 116.68 77.02)
+		(end 116.496 77.204)
+		(width 0.2)
+		(layer "B.Cu")
+		(net 1)
+	)
+	(segment
+		(start 116.330057 88.56)
+		(end 115.86 88.56)
+		(width 0.6)
+		(layer "B.Cu")
+		(net 1)
+	)
+	(segment
+		(start 106.144 88.396)
+		(end 106.14 88.4)
+		(width 0.2)
+		(layer "B.Cu")
+		(net 1)
+	)
+	(segment
+		(start 116.496 82.142)
+		(end 116.496 88.394057)
+		(width 1.5)
+		(layer "B.Cu")
+		(net 1)
+	)
+	(segment
+		(start 116.496 75.741)
+		(end 106.144 75.741)
+		(width 1.5)
+		(layer "B.Cu")
+		(net 1)
+	)
+	(segment
+		(start 106.144 88.543)
+		(end 114.92 88.543)
+		(width 1.5)
+		(layer "B.Cu")
+		(net 1)
+	)
+	(segment
+		(start 116.496 82.142)
+		(end 116.496 75.741)
+		(width 1.5)
+		(layer "B.Cu")
+		(net 1)
+	)
+	(segment
+		(start 116.496 77.204)
+		(end 116.496 82.142)
+		(width 1.5)
+		(layer "B.Cu")
+		(net 1)
+	)
+	(segment
+		(start 106.144 75.741)
+		(end 106.144 88.396)
+		(width 1.5)
+		(layer "B.Cu")
+		(net 1)
+	)
