File: K9HZ_Antenna_Tuner/K9HZ_Antenna_Tuner_KiCad_Projects/K9HZ_Antenna_Tuner_RF_Board_Project/K9HZ_Antenna_Tuner_RF_Board.kicad_sch (KiCad schematic)
At the start: 52 parts, among them J1 Conn_Coaxial, J2 Conn_Coaxial, J3 Conn_01x01_Pin, J4 Conn_01x01_Pin, J5 1986717-8, J6 1986717-8_8, J7 1986717-8_8, K1 HF41F_12-ZS, K10 HF41F_12-ZS, K11 HF41F_12-ZS, K12 HF41F_12-ZS, K13 HF41F_12-ZS, K14 HF41F_12-ZS, K15 HF41F_12-ZS, K16 HF41F_12-ZS, K17 HF41F_12-ZS, K18 HF41F_12-ZS, K19 HF41F_12-ZS, K2 HF41F_12-ZS, K20 HF41F_12-ZS, K3 HF41F_12-ZS, K4 HF41F_12-ZS, K5 HF41F_12-ZS, K6 HF41F_12-ZS, K7 HF41F_12-ZS, K8 HF41F_12-ZS, K9 HF41F_12-ZS, T1 Transformer_SP_1S

Commit message: Tuner Update
Tuner Update
Other:
- note added: "FOR"
- note added: "GND"
- note added: "OPTIONAL LINE SECTION: NOT USED FOR T41 WITH K9HZ LPF LINE SECTION"
- note added: "REF"
- note added: "RF IN"
- note added: "RF OUT"
- note removed: "POWER LINE SECTION"
Changed lines of the file:
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@@
 	(text "LC -CL"
 		(exclude_from_sim no)
-		(at 118.11 172.72 0)
+		(at 119.634 174.752 0)
 		(effects
 			(font
@@
 		)
 	)
+	(text "REF"
+		(exclude_from_sim no)
+		(at 71.12 88.9 0)
+		(effects
+			(font
+				(size 1.27 1.27)
+			)
+		)
+	)
 	(text "BN43-202"
 		(exclude_from_sim no)
@@
 		)
 	)
+	(text "RF IN"
+		(exclude_from_sim no)
+		(at 50.8 80.01 0)
+		(effects
+			(font
+				(size 1.27 1.27)
+			)
+		)
+	)
+	(text "RF OUT"
+		(exclude_from_sim no)
+		(at 71.12 80.01 0)
+		(effects
+			(font
+				(size 1.27 1.27)
+			)
+		)
+	)
 	(text "BALANCED OUT"
 		(exclude_from_sim no)
@@
 		)
 	)
+	(text "FOR"
+		(exclude_from_sim no)
+		(at 120.396 189.23 0)
+		(effects
+			(font
+				(size 1.48 1.48)
+			)
+		)
+	)
 	(text "BALANCED OUTPUT"
 		(exclude_from_sim no)
@@
 		)
 	)
-	(text "OPTIONAL LINE SECTION"
+	(text "GND"
 		(exclude_from_sim no)
-		(at 45.72 138.43 0)
+		(at 72.39 83.82 0)
+		(effects
+			(font
+				(size 1.27 1.27)
+			)
+		)
+	)
+	(text "OPTIONAL LINE SECTION:\nNOT USED FOR T41 WITH\nK9HZ LPF LINE SECTION"
+		(exclude_from_sim no)
+		(at 44.45 138.43 0)
 		(effects
 			(font
 				(size 1.48 1.48)
+				(color 0 0 255 1)
 			)
 			(justify left top)
@@
 		)
 	)
-	(text "POWER LINE SECTION"
+	(text "FOR"
 		(exclude_from_sim no)
-		(at 78.74 63.5 0)
+		(at 50.8 88.9 0)
 		(effects
 			(font
-				(size 2.467 2.467)
+				(size 1.27 1.27)
+			)
+		)
+	)
+	(text "OPTIONAL LINE SECTION"
+		(exclude_from_sim no)
+		(at 77.47 58.42 0)
+		(effects
+			(font
+				(size 2.032 2.032)
+				(thickness 0.4934)
+				(bold yes)
 			)
 			(justify right top)
@@
 	(text "BYPASS"
 		(exclude_from_sim no)
-		(at 111.76 179.07 0)
+		(at 114.808 179.07 0)
 		(effects
 			(font
@@
 		)
 	)
+	(text "REF"
+		(exclude_from_sim no)
+		(at 120.396 192.278 0)
+		(effects
+			(font
+				(size 1.48 1.48)
+			)
+		)
+	)
 	(text "J5"
 		(exclude_from_sim no)
@@
 	)
 	(junction
-		(at 44.45 104.14)
-		(diameter 0)
-		(color 0 0 0 0)
-	)
-	(junction
 		(at 328.93 22.86)
 		(diameter 0)
@@
 	(junction
 		(at 223.52 128.27)
+		(diameter 0)
+		(color 0 0 0 0)
+	)
+	(junction
+		(at 43.18 104.14)
 		(diameter 0)
 		(color 0 0 0 0)
@@
 	(wire
 		(pts
-			(xy 49.53 104.14) (xy 44.45 104.14)
-		)
-		(stroke
-			(width 0.25)
-			(type solid)
-		)
-	)
-	(wire
-		(pts
 			(xy 328.93 27.94) (xy 328.93 43.18)
 		)
@@
 	(wire
 		(pts
+			(xy 43.18 104.14) (xy 49.53 104.14)
+		)
+		(stroke
+			(width 0.25)
+			(type solid)
+		)
+	)
+	(wire
+		(pts
 			(xy 219.71 93.98) (xy 234.95 93.98)
 		)
@@
 	(wire
 		(pts
-			(xy 44.45 104.14) (xy 43.18 104.14)
-		)
-		(stroke
-			(width 0.25)
-			(type solid)
-		)
-	)
-	(wire
-		(pts
 			(xy 331.47 128.27) (xy 335.28 128.27)
 		)
@@
 	(wire
 		(pts
-			(xy 44.45 190.5) (xy 149.86 190.5)
+			(xy 43.18 190.5) (xy 149.86 190.5)
 		)
 		(stroke
@@
 	(wire
 		(pts
-			(xy 74.93 194.31) (xy 73.66 194.31)
+			(xy 73.66 193.04) (xy 149.86 193.04)
 		)
 		(stroke
@@
 	(wire
 		(pts
-			(xy 73.66 194.31) (xy 73.66 153.67)
-		)
-		(stroke
-			(width 0)
-			(type default)
-		)
-	)
-	(wire
-		(pts
-			(xy 149.86 193.04) (xy 74.93 193.04)
+			(xy 73.66 193.04) (xy 73.66 153.67)
 		)
 		(stroke
@@
 	(wire
 		(pts
-			(xy 44.45 104.14) (xy 44.45 190.5)
+			(xy 43.18 104.14) (xy 43.18 190.5)
 		)
 		(stroke
@@
 		)
 		(stroke
-			(width 0)
-			(type default)
-		)
-	)
-	(wire
-		(pts
-			(xy 74.93 194.31) (xy 74.93 193.04)
-		)
-		(stroke
