File: K9HZ_Antenna_Tuner/K9HZ_Antenna_Tuner_KiCad_Projects/K9HZ_Antenna_Tuner_RF_Board_Project/K9HZ_Antenna_Tuner_RF_Board.kicad_pcb (KiCad board)
At the start: 2 copper layers, 100 x 100 mm, 52 parts, among them J1 Conn_Coaxial, J2 Conn_Coaxial, J3 Conn_01x01_Pin, J4 Conn_01x01_Pin, J5 1986717-8, J6 1986717-8_8, J7 1986717-8_8, K1 HF41F_12-ZS, K10 HF41F_12-ZS, K11 HF41F_12-ZS, K12 HF41F_12-ZS, K13 HF41F_12-ZS, K14 HF41F_12-ZS, K15 HF41F_12-ZS, K16 HF41F_12-ZS, K17 HF41F_12-ZS, K18 HF41F_12-ZS, K19 HF41F_12-ZS, K2 HF41F_12-ZS, K20 HF41F_12-ZS, K3 HF41F_12-ZS, K4 HF41F_12-ZS, K5 HF41F_12-ZS, K6 HF41F_12-ZS, K7 HF41F_12-ZS, K8 HF41F_12-ZS, K9 HF41F_12-ZS, T1 Transformer_SP_1S

Commit message: Tuner Update
Tuner Update
Parts:
- added ?: , , F.Cu at (116.2, 109.6)
- moved K1 69.6 mm to (152.1, 51.9)
- moved K8 68.9 mm to (141.3, 85.6)
- moved C5 68.7 mm to (138.3, 144.5)
- moved J2 68.7 mm to (187.7, 90.5)
- moved C4 68.7 mm to (129.3, 145.9)
- moved C9 68.7 mm to (161.1, 143.9)
- moved H2 68.7 mm to (159.3, 61.7)
- moved H4 68.7 mm to (159.3, 135.7)
- moved J5 68.7 mm to (146.5, 66.7)
- moved J6 68.7 mm to (146.5, 91.3)
- moved J7 68.7 mm to (146.5, 115.9)
- moved L3 68.7 mm to (154.3, 90.1)
- moved L8 68.7 mm to (134.3, 99.3)
- moved C1 68.7 mm to (105.9, 145.9)
- moved C2 68.7 mm to (113.7, 145.9)
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Connections:
- L44 pad 1: Net-(J1-In) -> Net-(J7-P8)
- L44 pad 2: Net-(K19-COM) -> GND
- L44 pad 3: unconnected-(L44-COM-Pad3) -> Net-(J1-In)
- L44 pad 4: Net-(J7-P8) -> Net-(K19-COM)
Routing:
- net Net-(J7-P8): track 60.7 -> 90.7 mm, vias 0 -> 2
- net GND: track 28.5 -> 0.38 mm, vias 0 -> 6
- net Net-(J1-In): track 31.4 -> 38.1 mm
- net Net-(K17-NC): track 101.6 -> 107.6 mm
- net Net-(K5-NC): track 122.4 -> 126.3 mm
- net Net-(K6-NC): track 41.1 -> 44.8 mm
- net Net-(K19-COM): track 19.7 -> 22.9 mm
- net Net-(K19-NC): track 88.1 -> 89.5 mm
- net Net-(K17-COM): track 143.4 -> 142.4 mm
- net /K8.2: track 11.1 -> 10.0 mm
- net Net-(K1-NC): track 22.2 -> 21.7 mm
Other:
- board text added: "Copyright (C) 2026"
- board text added: "RF BOARD Version V2.0"
- board text added: "RF IN"
- board text added: "RF OUT"
- board text removed: "Copyright 2026"
- board text removed: "Generic Version V1.0"

Commit message: Tuner Update
Tuner Update
Parts:
- moved R1 1.97 mm to (99.8, 117.9)
Routing:
- net Net-(J7-P8): track 90.7 -> 92.7 mm
Changed lines of the file:
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@@
 	(footprint "Resistor_SMD:R_1206_3216Metric_Pad1.30x1.75mm_HandSolder"
 		(layer "F.Cu")
-		(at 101.7282 117.52 90)
+		(at 99.8 117.925 90)
 		(descr "Resistor SMD 1206 (3216 Metric), square (rectangular) end terminal, IPC-7351 nominal with elongated pad for handsoldering. (Body size source: IPC-SM-782 page 72, https://www.pcb-3d.com/wordpress/wp-content/uploads/ipc-sm-782a_amendment_1_and_2.pdf), generated with kicad-footprint-generator")
 		(tags "resistor handsolder")
@@
 	)
 	(via
-		(at 101.7282 119.07)
+		(at 99.8 119.475)
 		(size 0.6)
 		(drill 0.3)
@@
 	)
 	(segment
-		(start 101.7282 115.97)
-		(end 101.7282 99.948)
+		(start 101.7282 115.85)
+		(end 101.7 115.85)
+		(width 0.2)
+		(layer "F.Cu")
+		(net 27)
+	)
+	(segment
+		(start 101.7 115.85)
+		(end 101.175 116.375)
 		(width 0.2)
 		(layer "F.Cu")
@@
 		(width 0.2)
 		(layer "F.Cu")
+		(net 27)
+	)
+	(segment
+		(start 101.175 116.375)
+		(end 99.8 116.375)
+		(width 0.2)
+		(layer "F.Cu")
+		(net 27)
+	)
+	(segment
+		(start 101.7282 115.85)
+		(end 101.7282 99.948)
+		(width 0.2)
+		(layer "F.Cu")

Commit message: Update Tuner
Update Tuner for Production
Parts:
- added ?: , , F.Cu at (127.9, 100.8)
- moved L1 0.78 mm to (158.2, 68.8)
- moved L2 0.61 mm to (158.5, 76.6)
Routing:
- net /K17.1: track 48.4 -> 55.9 mm
- net /K12.1: track 23.8 -> 29.1 mm
- net /K11.1: track 34.2 -> 38.5 mm
- net /K10.1: track 43.8 -> 48.0 mm
- net /K9.1: track 53.8 -> 57.6 mm
- net /Bypass: track 96.3 -> 99.9 mm
- net /K13.1: track 16.1 -> 18.3 mm
- net Net-(K1-COM): track 76.8 -> 76.0 mm
- net Net-(K17-NC): track 107.6 -> 108.3 mm
